Commit message: 为机器人添加碰撞属性

File: chapt6/install/fishbot_description/share/fishbot_description/urdf/fishbot/actuator/caster.urdf.xacro (robot description, xacro)
@@ -16,4 +16,17 @@
                 </material>
             </visual>
+            <!-- 碰撞属性 -->
+            <collision>
+                <!-- 沿着自己几何中心的偏移和旋转 -->
+                <origin xyz="0.0 0.0 0.0" rpy="1.0 0.0 0.0"/>
+                <!-- 几何形状 -->
+                <geometry>
+                    <sphere radius="0.016"/>
+                </geometry>
+                <!-- 材质颜色 -->
+                <material name="yellow">
+                    <color rgba="1.0 1.0 0.0 0.8"/>
+                </material>
+            </collision>
         </link>
         <!-- 机器人的关节，用于组合机器人的部件 -->

File: chapt6/install/fishbot_description/share/fishbot_description/urdf/fishbot/actuator/wheel.urdf.xacro (robot description, xacro)
@@ -16,4 +16,17 @@
                 </material>
             </visual>
+            <!-- 碰撞属性 -->
+            <collision>
+                <!-- 沿着自己几何中心的偏移和旋转 -->
+                <origin xyz="0.0 0.0 0.0" rpy="1.57079 0.0 0.0"/>
+                <!-- 几何形状 -->
+                <geometry>
+                    <cylinder radius="0.032" length="0.04"/>
+                </geometry>
+                <!-- 材质颜色 -->
+                <material name="yellow">
+                    <color rgba="1.0 1.0 0.0 0.8"/>
+                </material>
+            </collision>
         </link>
         <!-- 机器人的关节，用于组合机器人的部件 -->

File: chapt6/install/fishbot_description/share/fishbot_description/urdf/fishbot/base.urdf.xacro (robot description, xacro)
@@ -19,4 +19,18 @@
                 </material>
             </visual>
+            <!-- 碰撞属性 -->
+            <collision>
+                <!-- 沿着自己几何中心的偏移和旋转 -->
+                <origin xyz="0.0 0.0 0.0" rpy="0.0 0.0 0.0"/>
+                <!-- 几何形状 -->
+                <geometry>
+                    <!-- 圆柱体 半径 0.10m 高度 0.12m -->
+                    <cylinder radius="${radius}" length="${length}"/>
+                </geometry>
+                <!-- 材质颜色 -->
+                <material name="white">
+                    <color rgba="1.0 1.0 1.0 0.5"/>
+                </material>
+            </collision>
         </link>
         <joint name="joint_name" type="fixed">

File: chapt6/install/fishbot_description/share/fishbot_description/urdf/fishbot/sensor/camera.urdf.xacro (robot description, xacro)
@@ -16,4 +16,17 @@
                 </material>
             </visual>
+            <!-- 碰撞属性 -->
+            <collision>
+                <!-- 沿着自己几何中心的偏移和旋转 -->
+                <origin xyz="0.0 0.0 0.0" rpy="0.0 0.0 0.0"/>
+                <!-- 几何形状 -->
+                <geometry>
+                    <box size="0.02 0.10 0.02"/>
+                </geometry>
+                <!-- 材质颜色 -->
+                <material name="black">
+                    <color rgba="0.0 0.0 0.0 0.5"/>
+                </material>
+            </collision>
         </link>
         <!-- 机器人的关节，用于组合机器人的部件 -->

File: chapt6/install/fishbot_description/share/fishbot_description/urdf/fishbot/sensor/laser.urdf.xacro (robot description, xacro)
@@ -34,4 +34,17 @@
                 </material>
             </visual>
+            <!-- 碰撞属性 -->
+            <collision>
+                <!-- 沿着自己几何中心的偏移和旋转 -->
+                <origin xyz="0.0 0.0 0.0" rpy="0.0 0.0 0.0"/>
+                <!-- 几何形状 -->
+                <geometry>
+                    <cylinder radius="0.02" length="0.02"/>
+                </geometry>
+                <!-- 材质颜色 -->
+                <material name="black">
+                    <color rgba="0.0 0.0 0.0 1.0"/>
+                </material>
+            </collision>
         </link>
         <!-- 机器人的关节，用于组合机器人的部件 -->

Commit message: 为机器人部件添加质量与惯性

File: chapt6/install/fishbot_description/share/fishbot_description/urdf/fishbot/actuator/caster.urdf.xacro (robot description, xacro)
@@ -1,4 +1,5 @@
 <?xml version="1.0"?>
 <robot xmlns:xacro="http://www.ros.org/wiki/xacro">
+<xacro:include filename="$(find fishbot_description)/urdf/fishbot/common_inertial.xacro"/>
     <xacro:macro name="caster_xacro" params="caster_name xyz">
         <link name="${caster_name}_link">
@@ -29,4 +30,5 @@
                 </material>
             </collision>
+            <xacro:sphere_inertia m="0.05" r="0.016" />
         </link>
         <!-- 机器人的关节，用于组合机器人的部件 -->

File: chapt6/install/fishbot_description/share/fishbot_description/urdf/fishbot/actuator/wheel.urdf.xacro (robot description, xacro)
@@ -1,4 +1,5 @@
 <?xml version="1.0"?>
 <robot xmlns:xacro="http://www.ros.org/wiki/xacro">
+<xacro:include filename="$(find fishbot_description)/urdf/fishbot/common_inertial.xacro"/>
     <xacro:macro name="wheel_xacro" params="wheel_name xyz">
         <link name="${wheel_name}_link">
@@ -29,4 +30,5 @@
                 </material>
             </collision>
+            <xacro:cylinder_inertia m="0.05" r="0.032" h="0.04" />
         </link>
         <!-- 机器人的关节，用于组合机器人的部件 -->

File: chapt6/install/fishbot_description/share/fishbot_description/urdf/fishbot/base.urdf.xacro (robot description, xacro)
@@ -1,4 +1,5 @@
 <?xml version="1.0"?>
 <robot xmlns:xacro="http://www.ros.org/wiki/xacro">
+<xacro:include filename="$(find fishbot_description)/urdf/fishbot/common_inertial.xacro"/>
     <xacro:macro name="base_xacro" params="length radius">
         <link name="base_footprint"/>
@@ -33,4 +34,5 @@
                 </material>
             </collision>
+            <xacro:cylinder_inertia m="1.0" r="${radius}" h="${length}" />
         </link>
         <joint name="joint_name" type="fixed">

File: chapt6/install/fishbot_description/share/fishbot_description/urdf/fishbot/sensor/camera.urdf.xacro (robot description, xacro)
@@ -1,4 +1,5 @@
 <?xml version="1.0"?>
 <robot xmlns:xacro="http://www.ros.org/wiki/xacro">
+<xacro:include filename="$(find fishbot_description)/urdf/fishbot/common_inertial.xacro"/>
     <xacro:macro name="camera_xacro" params="xyz">
         <link name="camera_link">
@@ -29,4 +30,5 @@
                 </material>
             </collision>
+            <xacro:box_inertia m="0.1" w="0.02" h="0.10" d="0.02" />
         </link>
         <!-- 机器人的关节，用于组合机器人的部件 -->

File: chapt6/install/fishbot_description/share/fishbot_description/urdf/fishbot/sensor/imu.urdf.xacro (robot description, xacro)
@@ -1,4 +1,5 @@
 <?xml version="1.0"?>
 <robot xmlns:xacro="http://www.ros.org/wiki/xacro">
+<xacro:include filename="$(find fishbot_description)/urdf/fishbot/common_inertial.xacro"/>
     <xacro:macro name="imu_xacro" params="xyz">
         <!-- 机器人的IMU部件，惯性测量传感器 -->
@@ -17,4 +18,18 @@
                 </material>
             </visual>
+            <!-- 碰撞属性 -->
+            <collision>
+                <!-- 沿着自己几何中心的偏移和旋转 -->
+                <origin xyz="0.0 0.0 0.0" rpy="0.0 0.0 0.0"/>
+                <!-- 几何形状 -->
+                <geometry>
+                    <box size="0.02 0.02 0.02"/>
+                </geometry>
+                <!-- 材质颜色 -->
+                <material name="black">
+                    <color rgba="0.0 0.0 0.0 0.5"/>
+                </material>
+            </collision>
+            <xacro:box_inertia m="0.05" w="0.02" h="0.02" d="0.02" />
         </link>
         <!-- 机器人的关节，用于组合机器人的部件 -->

File: chapt6/install/fishbot_description/share/fishbot_description/urdf/fishbot/sensor/laser.urdf.xacro (robot description, xacro)
@@ -1,4 +1,5 @@
 <?xml version="1.0"?>
 <robot xmlns:xacro="http://www.ros.org/wiki/xacro">
+<xacro:include filename="$(find fishbot_description)/urdf/fishbot/common_inertial.xacro"/>
     <xacro:macro name="laser_xacro" params="xyz">
         <!-- 雷达支撑杆 -->
@@ -18,4 +19,19 @@
                 </material>
             </visual>
+            <!-- 碰撞属性 -->
+            <collision>
+                <!-- 沿着自己几何中心的偏移和旋转 -->
+                <origin xyz="0.0 0.0 0.0" rpy="0.0 0.0 0.0"/>
+                <!-- 几何形状 -->
+                <geometry>
+                    <!-- 圆柱体 -->
+                    <cylinder radius="0.01" length="0.10"/>
+                </geometry>
+                <!-- 材质颜色 -->
+                <material name="black">
+                    <color rgba="0.0 0.0 0.0 1.0"/>
+                </material>
+            </collision>
+            <xacro:cylinder_inertia m="0.05" r="0.01" h="0.10" />
         </link>
         <!-- 雷达 -->
@@ -47,4 +63,5 @@
                 </material>
             </collision>
+            <xacro:cylinder_inertia m="0.10" r="0.02" h="0.02" />
         </link>
         <!-- 机器人的关节，用于组合机器人的部件 -->

Commit message: 使用gazebo标签扩展urdf

File: chapt6/install/fishbot_description/share/fishbot_description/urdf/fishbot/actuator/caster.urdf.xacro (robot description, xacro)
@@ -38,4 +38,15 @@
             <origin xyz="${xyz}" rpy="0.0 0.0 0.0"/>
         </joint>
+        <!-- 使用gazebo标签设置摩擦力 -->
+        <gazebo reference="${caster_name}_link">
+            <!-- 切向摩擦系数 -->
+            <mu1 value="0.0"/>
+            <!-- 法向摩擦系数 -->
+            <mu2 value="0.0"/>
+            <!-- 接触的刚度字数系数 -->
+            <kp value="1000000000.0"/>
+            <!-- 阻尼系数 -->
+            <kd value="1.0"/>
+        </gazebo>
     </xacro:macro>
 </robot>

File: chapt6/install/fishbot_description/share/fishbot_description/urdf/fishbot/actuator/wheel.urdf.xacro (robot description, xacro)
@@ -39,4 +39,15 @@
             <axis xyz="0.0 1.0 0.0"/>
         </joint>
+        <!-- 使用gazebo标签设置摩擦力 -->
+        <gazebo reference="${wheel_name}_link">
+            <!-- 切向摩擦系数 -->
+            <mu1 value="20.0"/>
+            <!-- 法向摩擦系数 -->
+            <mu2 value="20.0"/>
+            <!-- 接触的刚度字数系数 -->
+            <kp value="1000000000.0"/>
+            <!-- 阻尼系数 -->
+            <kd value="1.0"/>
+        </gazebo>
     </xacro:macro>
 </robot>

File: chapt6/install/fishbot_description/share/fishbot_description/urdf/fishbot/sensor/laser.urdf.xacro (robot description, xacro)
@@ -76,4 +76,11 @@
             <origin xyz="${xyz}" rpy="0.0 0.0 0.0"/>
         </joint>
+        <!-- gazebo标签，设置gazebo中的颜色 -->
+        <gazebo reference="laser_cylinder_link">
+            <material>Gazebo/Black</material>
+        </gazebo>
+        <gazebo reference="laser_link">
+            <material>Gazebo/Black</material>
+        </gazebo>
     </xacro:macro>
 </robot>
